Commit message: Updated urdf.
Signed-off-by: Benjamin Perseghetti <bperseghetti@rudislabs.com>

File: urdf/mrb3.urdf (robot description, URDF)
Before this commit: robot mrb3s, 2 links, 1 joints
Links:
- removed link mrb3s/RPLIDAR_A1M8/Base/lidar
- removed link mrb3s/base_footprint
- added link base_footprint
- added link base_laser; visual mesh filename=package://mrb3_description/meshes/rplidar.dae scale=1 1 1
- added link base_link; visual mesh filename=package://mrb3_description/meshes/MRB3.dae scale=1 1 1; visual mesh filename=package://mrb3_description/meshes/Wheel.dae scale=1 1 1
Joints:
- removed joint Joint
- added joint base_joint: type fixed, parent base_footprint, child base_link, origin xyz=0.0 0.0 0.0 rpy=0 0 0
- added joint laser_joint: type fixed, parent base_link, child base_laser, origin xyz=0.042 0 0.096 rpy=0 0 0
